Commit message: Refactor: Servidor modularizado, soporte asíncrono para ROS2 y renderizado LaTeX

File: src/lynx_al5d_ros2_description/urdf/lynx_al5d.urdf.xacro (robot description, xacro)
@@ -4,6 +4,5 @@
     <xacro:property name="mesh_path" value="package://${package_name}/meshes/robot_parts/"/>
     <xacro:property name="PI" value="3.1415926535897931"/>
-    <xacro:property name="shoulder_to_elbow" value="0.146" />
-    <xacro:property name="tube_length" value="0.15" />
+    <xacro:property name="altura_base" value="0.115" />       <xacro:property name="shoulder_to_elbow" value="0.155" /> <xacro:property name="elbow_to_wrist" value="0.185" />    <xacro:property name="tube_length" value="0.15" />
     <xacro:property name="hs_755eb_depth" value="0.05" />
     <xacro:property name="gripper_base_width" value="0.03175" />
@@ -138,5 +137,5 @@
         <child link="shoulder_link" />
         <axis xyz="1 0 0"/>
-        <origin xyz="0 0.02 0.07" />
+        <origin xyz="0 0.02 ${altura_base}" />
         <limit effort="100" velocity="3" lower="0" upper="${PI}" />
     </joint>
@@ -152,5 +151,5 @@
         <child link="wrist_link" />
         <axis xyz="1 0 0" />
-        <origin xyz="0 0.181 0.005" rpy="0 0 0"/>
+        <origin xyz="0 ${elbow_to_wrist} 0.005" rpy="0 0 0"/>
         <limit effort="40" velocity="3" lower="${-PI/2}" upper="${PI/2}" />
     </joint>
@@ -168,5 +167,4 @@
         <axis xyz="-1 0 0" />
         <limit effort="100" velocity="0.1" lower="0" upper="${gripper_base_width/2}" />
-        <dynamics damping="1.0" friction="0.16" />
     </joint>
     <joint name="joint_gripper_left_finger" type="prismatic">
@@ -177,39 +175,4 @@
         <mimic joint="joint_gripper_finger" multiplier="1.0" offset="0" />
         <limit effort="100" velocity="0.1" lower="0" upper="${gripper_base_width/2}" />
-        <dynamics damping="1.0" friction="0.16" />
     </joint>
-    <ros2_control name="GazeboSystem" type="system">
-        <hardware>
-            <plugin>gazebo_ros2_control/GazeboSystem</plugin>
-        </hardware>
-        <joint name="joint_base_rotate">
-            <command_interface name="position"/>
-            <state_interface name="position"/>
-        </joint>
-        <joint name="joint_shoulder">
-            <command_interface name="position"/>
-            <state_interface name="position"/>
-        </joint>
-        <joint name="joint_elbow">
-            <command_interface name="position"/>
-            <state_interface name="position"/>
-        </joint>
-        <joint name="joint_wrist">
-            <command_interface name="position"/>
-            <state_interface name="position"/>
-        </joint>
-        <joint name="joint_gripper_rotate">
-            <command_interface name="position"/>
-            <state_interface name="position"/>
-        </joint>
-        <joint name="joint_gripper_finger">
-            <command_interface name="position"/>
-            <state_interface name="position"/>
-        </joint>
-    </ros2_control>
-    <gazebo>
-        <plugin name="gazebo_ros2_control" filename="libgazebo_ros2_control.so">
-            <parameters>$(find ${package_name})/config/robot_control.yaml</parameters>
-        </plugin>
-    </gazebo>
 </robot>
